File: MultiMediaSystem/AudioAmp/AudioAmp.kicad_pcb (KiCad board)
At the start: 4 copper layers, 85.6 x 64.5 mm, 61 parts, among them J1 Ctrl_pins, J2 PWR, J3 AudioIn, J4 PULLUP_SRC, J5 Rspkr_o, J6 Lspkr_o, Q1 q, U1 TAS5412TPHDRQ1

Commit message: Adjusted Motherboard Pinouts
Motherboard pinout's were slightly off. This corrects that problem.
Parts:
- moved J6 2.58 mm to (179.7, 117.8), turned to 180 degrees
- moved J5 2.57 mm to (179.7, 109.2), turned to 180 degrees
Routing:
- net R_o-: track 22.5 -> 20.4 mm
- net L_o+: track 16.4 -> 15.3 mm
- net L_o-: track 16.5 -> 15.4 mm
- net R_o+: track 19.2 -> 18.7 mm
Changed lines of the file:
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@@
   )
   (footprint "Connector_PinHeader_2.54mm:PinHeader_1x02_P2.54mm_Vertical" (layer "F.Cu")
-    (at 179.7 106.66)
+    (at 179.69 109.23 180)
     (descr "Through hole straight pin header, 1x02, 2.54mm pitch, single row")
     (tags "Through hole pin header THT 1x02 2.54mm single row")
@@
     (fp_line (start -1.27 3.81) (end -1.27 -0.635) (layer "F.Fab") (width 0.1))
     (fp_line (start 1.27 3.81) (end -1.27 3.81) (layer "F.Fab") (width 0.1))
-    (pad "1" thru_hole rect (at 0 0) (size 1.7 1.7) (drill 1) (layers *.Cu *.Mask)
+    (pad "1" thru_hole rect (at 0 0 180) (size 1.7 1.7) (drill 1) (layers *.Cu *.Mask)
       (net 23 "R_o+") (pinfunction "Pin_1") (pintype "passive"))
-    (pad "2" thru_hole oval (at 0 2.54) (size 1.7 1.7) (drill 1) (layers *.Cu *.Mask)
+    (pad "2" thru_hole oval (at 0 2.54 180) (size 1.7 1.7) (drill 1) (layers *.Cu *.Mask)
       (net 22 "R_o-") (pinfunction "Pin_2") (pintype "passive"))
     (model "${KICAD6_3DMODEL_DIR}/Connector_PinHeader_2.54mm.3dshapes/PinHeader_1x02_P2.54mm_Vertical.wrl"
@@
   )
   (footprint "Connector_PinHeader_2.54mm:PinHeader_1x02_P2.54mm_Vertical" (layer "F.Cu")
-    (at 179.7 115.27)
+    (at 179.68 117.85 180)
     (descr "Through hole straight pin header, 1x02, 2.54mm pitch, single row")
     (tags "Through hole pin header THT 1x02 2.54mm single row")
@@
     (fp_line (start -0.635 -1.27) (end 1.27 -1.27) (layer "F.Fab") (width 0.1))
     (fp_line (start -1.27 -0.635) (end -0.635 -1.27) (layer "F.Fab") (width 0.1))
-    (pad "1" thru_hole rect (at 0 0) (size 1.7 1.7) (drill 1) (layers *.Cu *.Mask)
+    (pad "1" thru_hole rect (at 0 0 180) (size 1.7 1.7) (drill 1) (layers *.Cu *.Mask)
       (net 25 "L_o+") (pinfunction "Pin_1") (pintype "passive"))
-    (pad "2" thru_hole oval (at 0 2.54) (size 1.7 1.7) (drill 1) (layers *.Cu *.Mask)
+    (pad "2" thru_hole oval (at 0 2.54 180) (size 1.7 1.7) (drill 1) (layers *.Cu *.Mask)
       (net 24 "L_o-") (pinfunction "Pin_2") (pintype "passive"))
     (model "${KICAD6_3DMODEL_DIR}/Connector_PinHeader_2.54mm.3dshapes/PinHeader_1x02_P2.54mm_Vertical.wrl"
@@
   (segment (start 171.895 103.955) (end 172.22 103.63) (width 1) (layer "F.Cu") (net 22))
   (segment (start 166.3 97.19) (end 168.09 97.19) (width 1) (layer "F.Cu") (net 22))
+  (segment (start 176.63 103.63) (end 179.69 106.69) (width 1) (layer "F.Cu") (net 22))
   (segment (start 169.595 103.48) (end 170.07 103.955) (width 1) (layer "F.Cu") (net 22))
   (segment (start 168.09 97.19) (end 169.595 98.695) (width 1) (layer "F.Cu") (net 22))
   (segment (start 170.07 103.955) (end 171.895 103.955) (width 1) (layer "F.Cu") (net 22))
+  (segment (start 175.195 103.63) (end 176.63 103.63) (width 1) (layer "F.Cu") (net 22))
   (segment (start 169.595 98.695) (end 169.595 103.48) (width 1) (layer "F.Cu") (net 22))
-  (segment (start 179.7 109.2) (end 178.9 109.2) (width 1) (layer "B.Cu") (net 22))
-  (segment (start 178.9 109.2) (end 175.195 105.495) (width 1) (layer "B.Cu") (net 22))
-  (segment (start 175.195 105.495) (end 175.195 104.865) (width 1) (layer "B.Cu") (net 22))
-  (segment (start 175.195 104.865) (end 175.195 103.63) (width 1) (layer "B.Cu") (net 22))
-  (segment (start 175.195 108.63) (end 177.165 106.66) (width 1) (layer "F.Cu") (net 23))
   (segment (start 166.3 108.2) (end 167.4 109.3) (width 1) (layer "F.Cu") (net 23))
-  (segment (start 177.165 106.66) (end 179.7 106.66) (width 1) (layer "F.Cu") (net 23))
   (segment (start 167.4 109.3) (end 169.595 109.3) (width 1) (layer "F.Cu") (net 23))
   (segment (start 166.3 103.9) (end 166.3 108.2) (width 1) (layer "F.Cu") (net 23))
   (segment (start 172.17 108.63) (end 175.195 108.63) (width 1) (layer "F.Cu") (net 23))
+  (segment (start 175.795 109.23) (end 175.195 108.63) (width 1) (layer "F.Cu") (net 23))
+  (segment (start 179.69 109.23) (end 175.795 109.23) (width 1) (layer "F.Cu") (net 23))
   (segment (start 171.5 109.3) (end 172.17 108.63) (width 1) (layer "F.Cu") (net 23))
   (segment (start 169.595 109.3) (end 171.5 109.3) (width 1) (layer "F.Cu") (net 23))
@@
   (segment (start 170.975 114.1) (end 170.9 114.025) (width 0.2) (layer "F.Cu") (net 24))
   (segment (start 170.525 113.55) (end 170.9 113.925) (width 1) (layer "F.Cu") (net 24))
+  (segment (start 177.83 115.27) (end 176.66 114.1) (width 1) (layer "F.Cu") (net 24))
+  (segment (start 177.83 115.27) (end 179.7 115.27) (width 1) (layer "F.Cu") (net 24))
   (segment (start 168.7 113.55) (end 170.525 113.55) (width 1) (layer "F.Cu") (net 24))
   (segment (start 170.9 113.925) (end 171.075 114.1) (width 0.2) (layer "F.Cu") (net 24))
   (segment (start 165.23 113.245) (end 168.395 113.245) (width 1) (layer "F.Cu") (net 24))
   (segment (start 168.395 113.245) (end 168.7 113.55) (width 0.75) (layer "F.Cu") (net 24))
-  (segment (start 174 114.1) (end 177.71 117.81) (width 1) (layer "B.Cu") (net 24))
-  (segment (start 177.71 117.81) (end 179.7 117.81) (width 1) (layer "B.Cu") (net 24))
+  (segment (start 176.66 114.1) (end 174 114.1) (width 1) (layer "F.Cu") (net 24))
+  (segment (start 178.43 119.1) (end 179.68 117.85) (width 1) (layer "F.Cu") (net 25))
   (segment (start 171.275 119.1) (end 174 119.1) (width 1) (layer "F.Cu") (net 25))
   (segment (start 170.9 119.475) (end 171.275 119.1) (width 0.2) (layer "F.Cu") (net 25))
   (segment (start 165.23 119.955) (end 168.595 119.955) (width 1) (layer "F.Cu") (net 25))
   (segment (start 170.525 119.85) (end 170.9 119.475) (width 1) (layer "F.Cu") (net 25))
-  (segment (start 174 119.1) (end 177.83 115.27) (width 1) (layer "F.Cu") (net 25))
-  (segment (start 177.83 115.27) (end 179.7 115.27) (width 1) (layer "F.Cu") (net 25))
+  (segment (start 174 119.1) (end 178.43 119.1) (width 1) (layer "F.Cu") (net 25))
   (segment (start 168.595 119.955) (end 168.7 119.85) (width 0.75) (layer "F.Cu") (net 25))
   (segment (start 168.7 119.85) (end 170.525 119.85) (width 1) (layer "F.Cu") (net 25))

Commit message: Updated all designs
Parts:
- RV1: value R_Potentiometer -> 50K pot
Connections:
- J2 pad 1: GND -> +12V
- J2 pad 2: +12V -> GND
- J2 pad 3: GND -> +12V
- J2 pad 4: +12V -> GND
- J2 pad 5: GND -> +12V
- J2 pad 6: +12V -> GND
Routing:
- net GND: track 99.7 -> 130.1 mm
- net +12V: track 39.2 -> 38.2 mm
Other:
- board text added: "12V"
- board text added: "3.3V"
- board text added: "AGND"
- board text added: "CLIP"
- board text added: "FAULT"
- board text added: "GND"
- board text added: "L"
- board text added: "L+"
- board text added: "L-"
- board text added: "MUTE"
- board text added: "R"
- board text added: "R+"
- board text added: "R-"
- board text added: "SCL"
- board text added: "SDA"
- board text added: "STBY"
