File: MultiMediaSystem/AudioAmp/AudioAmp.kicad_sch (KiCad schematic)
At the start: 61 parts, among them J1 Ctrl_pins, J2 PWR, J3 AudioIn, J4 PULLUP_SRC, J5 Rspkr_o, J6 Lspkr_o, Q1 q, U1 TAS5412TPHDRQ1

Commit message: Updated all designs
Connections:
- net +12V: now also J2.1 (Pin_1), J2.3 (Pin_3), J2.5 (Pin_5), L1.2; no longer J2.2 (Pin_2), J2.4 (Pin_4), J2.6 (Pin_6), L1.1
- net GND: now also J2.2 (Pin_2), J2.4 (Pin_4), J2.6 (Pin_6), U1.EPAD; no longer J2.1 (Pin_1), J2.3 (Pin_3), J2.5 (Pin_5)
- net PVDD: now also L1.1; no longer L1.2
- no-connect marks 2 -> 1
Other:
- moved on the sheet: L1
