File: MultiMediaSystem/PS_controller/PS_controller.kicad_sch (KiCad schematic)
At the start: 22 parts, among them J1 PWR_IN, J2 serial, J3 FET_CTRL, J4 FET_CTRL, Q1 AO3401A, T1 TrinketPro_5V, U1 LT3970HMS-TRPBF

Commit message: Updated all designs
Parts:
- removed J2: serial, Connector_PinSocket_2.54mm:PinSocket_1x03_P2.54mm_Vertical, symbol Connector_Generic:Conn_01x03
- removed J3: FET_CTRL, Connector_PinSocket_2.54mm:PinSocket_1x02_P2.54mm_Vertical, symbol Connector_Generic:Conn_01x02
- added H3: MountingHole, MountingHole:MountingHole_2.5mm, symbol Mechanical:MountingHole
- added R1, R3: JMP, Resistor_SMD:R_0805_2012Metric_Pad1.20x1.40mm_HandSolder, symbol Device:R_Small
- added R10: 100K, Resistor_SMD:R_1206_3216Metric_Pad1.30x1.75mm_HandSolder, symbol Device:R_Small
- added R5: 1M, Resistor_SMD:R_0805_2012Metric_Pad1.20x1.40mm_HandSolder, symbol Device:R
- added R8: 316K, Resistor_SMD:R_1206_3216Metric_Pad1.30x1.75mm_HandSolder, symbol Device:R
- C1: value 2.2u -> 2.2uF
- R2: value CT6ER105_1M_282k -> 1M_Pot
- Rt1: footprint Resistor_SMD:R_0402_1005Metric_Pad0.72x0.64mm_HandSolder -> Resistor_SMD:R_0805_2012Metric_Pad1.20x1.40mm_HandSolder
- T1: footprint Arduino:TrinketPro5V -> Arduino:TrinketPro5V_partial
Connections:
- net +12V: now also Q1.3 (D), R1.1; no longer Q1.2 (D)
- net 5.5V: now also R2.3, R5.1; no longer R2.1
- net EN: now also R3.1
- net FB: now also C4.2, R5.2, R8.2
- net GND: now also R2.1, R10.1, R8.1; no longer C4.2, D1.2 (A), Q1.1 (G), R2.3
- net Vin: now also Q1.2 (S), R1.2, R3.2; no longer Q1.3 (S)
- net RELAY: no longer names the net of T1.3
- removed net UART_RX: T1.1 (RX)
- removed net UART_TX: T1.2 (TX)
- new net: D1.2 (A), Q1.1 (G), R10.2
- no-connect marks 16 -> 19
Other:
- note added: "FB voltage output: R1 = R2(Vout/1.21 -1)"
- note added: "Potentiometer R value = 1.03M Vout = 5.5V, R2 = R2 - R1 R1 = (Rt-R1)(Vout/1.21-1) R1 + R1(Vout/1.21-1) = Rt(Vout/1.21-1) R1(Vout/1.21)) = Rt(vout/1.21-1) R1 = 803.4K"
- note added: "Potentiometer Rt value = 20.29K Vin = 10-16V, Vout = 0-5V R1 = Rt-R2 Vout = Vin(R2/(R1+R2) Vin(R2/((Rt-R2)+R2) Vout*Rt/Vin = R2 100k/16 = R2 = 6.34K R1 = 13.95"
- moved on the sheet: C4, C5, D1, H1, H2, R2, R4, Rt1
