File: MultiMediaSystem/Regulator_5V/Regulator_5V.kicad_pcb (KiCad board)
At the start: 2 copper layers, 58.9 x 32.9 mm, 12 parts, among them J1 Conn_01x03, U1 TPS5450DDAR

Commit message: Updated all designs
Other:
- board text added: "Vin"
- board text added: "Vout"
Changed lines of the file:
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@@
   )
   (paper "A4")
+  (title_block
+    (title "5V Reg")
+    (date "2022-05-22")
+    (rev "1.1")
+  )
   (layers
     (0 "F.Cu" signal)
@@
     (property "Sheetname" "")
     (attr smd)
-    (fp_text reference "C3" (at 0 -1.778 180) (layer "F.SilkS") hide
+    (fp_text reference "C3" (at -0.1345 1.64 -90) (layer "F.SilkS")
       (effects (font (size 1 1) (thickness 0.15)))
     )
@@
       (effects (font (size 1 1) (thickness 0.15)))
     )
-    (fp_text value "Conn_01x03" (at 4.385 7.35 180) (layer "F.Fab")
+    (fp_text value "Conn_01x03" (at 9.475 2.025 180) (layer "F.Fab")
       (effects (font (size 1 1) (thickness 0.15)))
     )
@@
   )
   (gr_rect (start 127.9 71.9) (end 186.8 104.8) (layer "Edge.Cuts") (width 0.1) (fill none))
+  (gr_text "Vout" (at 132 74.1) (layer "F.SilkS")
+    (effects (font (size 1 1) (thickness 0.15)))
+  )
+  (gr_text "Vin" (at 132.1 84) (layer "F.SilkS")
+    (effects (font (size 1 1) (thickness 0.15)))
+  )
   (segment (start 138.9215 85.50685) (end 138.9215 85.0825) (width 0.25) (layer "F.Cu") (net 1))
   (segment (start 136.74235 87.686) (end 138.9215 85.50685) (width 0.5) (layer "F.Cu") (net 1))
