File: MultiMediaSystem/Regulator_5V/Regulator_5V.kicad_sch (KiCad schematic)
At the start: 12 parts, among them J1 Conn_01x03, U1 TPS5450DDAR

Commit message: Updated all designs
Parts:
- D1: footprint Diode_SMD:D_SMC-RM10_Universal_Handsoldering -> Diode_SMD:D_MELF_Handsoldering
Other:
- note added: "Output voltage setpoint: R1 = 10k, Vout = 5V R2 = R1*1.221/(Vout-1.221) R2 = 3231Kohm"
Changed lines of the file:
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@@
     (stroke (width 0) (type default) (color 0 0 0 0))
+  )
+  (text "Output voltage setpoint:\nR1 = 10k, Vout = 5V\nR2 = R1*1.221/(Vout-1.221)\nR2 = 3231Kohm"
+    (at 166.116 75.692 0)
+    (effects (font (size 1.27 1.27)) (justify left bottom))
   )
   (global_label "Boot" (shape input) (at 110.49 34.29 180) (fields_autoplaced)
@@
       (effects (font (size 1.27 1.27)) (justify left))
     )
-    (property "Footprint" "Diode_SMD:D_SMC-RM10_Universal_Handsoldering" (id 2) (at 128.27 38.1 0)
+    (property "Footprint" "Diode_SMD:D_MELF_Handsoldering" (id 2) (at 128.27 38.1 0)
       (effects (font (size 1.27 1.27)) hide)
     )
@@
     )
     (path "/5d24fc1f-7dba-462e-9cf0-f98c050d95e8"
-      (reference "D1") (unit 1) (value "B540C") (footprint "Diode_SMD:D_SMC-RM10_Universal_Handsoldering")
+      (reference "D1") (unit 1) (value "B540C") (footprint "Diode_SMD:D_MELF_Handsoldering")
     )
     (path "/42688fc6-3e24-4a56-9963-828da46dcdfb"
