File: MultiMediaSystem/StereoPS/StereoPS.kicad_pcb (KiCad board)
At the start: 2 copper layers, 98.5 x 51.3 mm, 30 parts, among them J1 PwrIn, J2 PwrOut, Q1 RX3G07CGNC16, Q2 RX3G07CGNC16, Q3 RX3G07CGNC16, Q4 RX3G07CGNC16, U1 LTC3780IG-PBF

Commit message: Updated all designs
Parts:
- Q1, Q2, Q3, Q4: footprint Package_TO_SOT_THT:TO-220-3_Horizontal_TabDown -> Custom:TO-220-3_Horizontal_TabDown_Thermal
Routing:
- net Vin: track 73.0 -> 114.7 mm
- net GND: track 66.3 -> 69.1 mm
- net TG2: track 37.5 -> 35.5 mm
