File: MultiMediaSystem/StereoPS/StereoPS.kicad_sch (KiCad schematic)
At the start: 30 parts, among them J1 PwrIn, J2 PwrOut, Q1 RX3G07CGNC16, Q2 RX3G07CGNC16, Q3 RX3G07CGNC16, Q4 RX3G07CGNC16, U1 LTC3780IG-PBF

Commit message: Updated all designs
Parts:
- removed J1: PwrIn, Custom:PinHeader_1x03_P2.54mm_Horizontal, symbol Connector_Generic:Conn_01x03
- removed U1: LTC3780IG-PBF, Imported:LTC3780IG-PBF, symbol Regulator_Switching:LTC3780IG-PBF
- added C10: 47pF, Capacitor_SMD:C_0603_1608Metric_Pad1.08x0.95mm_HandSolder, symbol Device:C_Small
- added C6: .1uF, Capacitor_SMD:C_0603_1608Metric_Pad1.08x0.95mm_HandSolder, symbol Device:C_Small
- added J1: PwrIn, Custom:PinHeader_1x02_P2.54mm_Horizontal, symbol Connector_Generic:Conn_01x02
- added J3: GND, Custom:PinHeader_1x02_P2.54mm_Horizontal, symbol Connector_Generic:Conn_01x02
- added J4: PGood, Connector_PinSocket_2.54mm:PinSocket_1x01_P2.54mm_Vertical, symbol Connector_Generic:Conn_01x01
- added J5: ExtVCC, Connector_PinSocket_2.54mm:PinSocket_1x01_P2.54mm_Vertical, symbol Connector_Generic:Conn_01x01
- added J6: CtrlPins, Connector_PinSocket_2.54mm:PinSocket_1x04_P2.54mm_Vertical, symbol Connector_Generic:Conn_01x04
- added R10, R7, R8, R9: JMP, Resistor_SMD:R_0805_2012Metric_Pad1.20x1.40mm_HandSolder, symbol Device:R_Small
- added R5: 49.9K, Resistor_SMD:R_0805_2012Metric_Pad1.20x1.40mm_HandSolder, symbol Device:R_Small
- added R6: 11K, Resistor_SMD:R_0805_2012Metric_Pad1.20x1.40mm_HandSolder, symbol Device:R_Small
- added U1: LTC3780IG-PBF, Imported:LTC3780IG-PBF, symbol Custom:LTC3780IG-PBF
- D1, D2: footprint Diode_SMD:D_MELF-RM10_Universal_Handsoldering -> Diode_SMD:D_MELF_Handsoldering
- L1: footprint Inductor_SMD:L_12x12mm_H8mm -> Inductor_Coilcraft:L_12x12mm_H8mm
- QA1: renamed from Q3; footprint Package_TO_SOT_THT:TO-220-3_Horizontal_TabDown -> Custom:TO-220-3_Horizontal_TabDown_Thermal; symbol Device:Q_NMOS_DGS -> Custom:Q_NMOS_DGS_THERMAL
- QB1: renamed from Q1; footprint Package_TO_SOT_THT:TO-220-3_Horizontal_TabDown -> Custom:TO-220-3_Horizontal_TabDown_Thermal; symbol Device:Q_NMOS_DGS -> Custom:Q_NMOS_DGS_THERMAL
- QC1: renamed from Q4; footprint Package_TO_SOT_THT:TO-220-3_Horizontal_TabDown -> Custom:TO-220-3_Horizontal_TabDown_Thermal; symbol Device:Q_NMOS_DGS -> Custom:Q_NMOS_DGS_THERMAL
- QD1: renamed from Q2; footprint Package_TO_SOT_THT:TO-220-3_Horizontal_TabDown -> Custom:TO-220-3_Horizontal_TabDown_Thermal; symbol Device:Q_NMOS_DGS -> Custom:Q_NMOS_DGS_THERMAL
- R2, R4: footprint Resistor_THT:R_Axial_DIN0414_L11.9mm_D4.5mm_P15.24mm_Horizontal -> Resistor_SMD:R_1206_3216Metric_Pad1.30x1.75mm_HandSolder
- R3: value 0Ohm -> Rpull; footprint Resistor_SMD:R_0402_1005Metric_Pad0.72x0.64mm_HandSolder -> Resistor_SMD:R_0805_2012Metric_Pad1.20x1.40mm_HandSolder
- renumbered C7 to CA1, C6 to CB1
Connections:
- net +12V: now also QA1.2 (D), J1.1 (Pin_1), J1.2 (Pin_2), R5.1, U1.21 (VIN); no longer QA1.1 (D)
- net BG1: now also QC1.1 (G), U1.18 (BG1); no longer QC1.2 (G)
- net BG2: now also QB1.1 (G), U1.16 (BG2); no longer QB1.2 (G)
- net Boost1: now also U1.24 (BOOST1)
- net Boost2: now also U1.13 (BOOST2)
- net FCB: now also R10.2, R9.2, U1.9 (FCB); no longer R3.2
- net GND: now also QA1.4 (EPAD), QB1.4 (EPAD), QC1.4 (EPAD), QD1.4 (EPAD), C10.2, C6.2, J3.1 (Pin_1), J3.2 (Pin_2), R6.2, R7.1, R8.1, R9.1, U1.17 (PGND), U1.4 (SENSE-), U1.7 (SGND); no longer R3.1
- net INTVCC: now also R10.1, U1.19 (INTVCC)
- net Ith: now also C10.1, U1.5 (ITH)
- net SENSE+: now also U1.3 (SENSE+)
- net SS: now also C6.1, U1.2 (SS); no longer C5.1
- net SW1: now also QC1.2 (D), U1.22 (SW1); no longer QC1.1 (D)
- net SW2: now also QB1.2 (D), U1.15 (SW2); no longer QB1.1 (D)
- net TG1: now also QD1.1 (G), U1.23 (TG1); no longer QD1.2 (G)
- net TG2: now also QA1.1 (G), U1.14 (TG2); no longer QA1.2 (G)
- net Vout: now also QD1.2 (D), R2.1; no longer QD1.1 (D), R2.2
- net Vsense: now also R2.2, U1.6 (VOSENSE); no longer R2.1
- new net: R3.2, U1.1 (PGOOD)
- new net EXTVCC: J5.1 (Pin_1), R7.2, U1.20 (EXTVCC)
- new net PGOOD: J4.1 (Pin_1), R3.1
- new net PLLFLTR: J6.3 (Pin_3), R8.2, U1.10 (PLLFLTR)
- new net PLLIN: J6.2 (Pin_2), U1.11 (PLLIN)
- new net RUN: J6.4 (Pin_4), R5.2, R6.1, U1.8 (RUN)
- new net STBYMD: C5.1, J6.1 (Pin_1), U1.12 (STBYMD)
- no-connect marks 6 -> 0
Other:
- note added: "EXTVCC tied to GND when not being used"
- note added: "FCB can be tied to one of three voltages for different ctrl modes GND for continuous operation Float for burst mode IntVcc for discontinuous current mode"
- note added: "Key Information: RUN Pin must be <6V EXTVCC: Source for internal voltage driver. Not needed and can be tied to gnd PLLIN: External Phase locked loop source, add a connector and leave alone PLLFLTR: Frequency selection. Leaving open will result in minimum frequency STBYMD: Used to provide wake up logic, un-needed, bypass to gnd"
- note added: "PLLFLTR only used when PLLIN being used. If PLLIN is open tie to GND"
- note added: "Run must be >2V and <6V at all times"
- note added: "STBYMD bypass to gnd when not used for control logic"
- note added: "Vout setpoint: Vout = .8*(1+R2/R1) R2 ~= 105k R1 = R2/(Vout/.8 - 1)"
- note added: "https://www.digikey.com/en/products/detail/yageo/RC0805FR-1310KL/13694107"
- moved on the sheet: C1, C2, C3, C4, C8, C9, CA1, CB1, D1, D2, DA1, DB1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
